File: Kicad/ADS131M08_Input.kicad_sch (KiCad schematic)
At the start: 60 parts, among them J2 Conn_02x10_Odd_Even, U3 ADS131M08, U4 LP5907MFX-3.3, X1 SIT8924BA

Commit message: Fix PCB Issues
Fix ADS131M08 Pinout
Fix ADS131M08 footprint size
Replace tiny ESD devices
Parts:
- removed D10, D11, D12, D13, D14, D15, D16, D17, D18, D19, D4, D5, D6, D7, D8, D9: PESD2V0Y1, Diode_SMD:D_SOD-923, symbol Diode:ESD9B3.3ST5G
- added D4, D5, D6, D7: ESDA6V1BC6, Package_TO_SOT_SMD:SOT-23-6, symbol Power_Protection:ESDA6V1BC6
- U3: footprint Package_QFP:TQFP-32_7x7mm_P0.8mm -> Package_QFP:PQFP-32_5x5mm_P0.5mm
Connections:
- net AIN1N: now also U3.31 (AIN1N); no longer U3.32 (AIN1N)
- net AIN1P: now also U3.32 (AIN1P); no longer U3.31 (AIN1P)
- net AIN3N: now also U3.3 (AIN3N); no longer U3.4 (AIN3N)
- net AIN3P: now also U3.4 (AIN3P); no longer U3.3 (AIN3P)
- net AIN5N: now also U3.7 (AIN5N); no longer U3.8 (AIN5N)
- net AIN5P: now also U3.8 (AIN5P); no longer U3.7 (AIN5P)
- net AIN7N: now also U3.11 (AIN7N); no longer U3.12 (AIN7N)
- net AIN7P: now also U3.12 (AIN7P); no longer U3.11 (AIN7P)
- net GND: now also D4.2 (COM), D4.5 (COM), D5.2 (COM), D5.5 (COM), D6.2 (COM), D6.5 (COM), D7.2 (COM), D7.5 (COM)
- net IN0N: now also D4.6 (TVS4)
- net IN0P: now also D4.1 (TVS1)
- net IN1N: now also D4.4 (TVS3)
- net IN1P: now also D4.3 (TVS2)
- net IN2N: now also D5.6 (TVS4)
- net IN2P: now also D5.1 (TVS1)
- net IN3N: now also D5.4 (TVS3)
- net IN3P: now also D5.3 (TVS2)
- net IN4N: now also D6.6 (TVS4)
- net IN4P: now also D6.1 (TVS1)
- net IN5N: now also D6.4 (TVS3)
- net IN5P: now also D6.3 (TVS2)
- net IN6N: now also D7.6 (TVS4)
- net IN6P: now also D7.1 (TVS1)
- net IN7N: now also D7.4 (TVS3)
- net IN7P: now also D7.3 (TVS2)
Other:
- note added: "ESDA6V1-4BC6 Quad Bidirectional ESD Protection according to IEC 61000-4-2 level 4 Reverse Standoff Voltage = 1uA @ 3V Breakdown Voltage max = 8V Capacitance 45pF Leakage current max = 1uA"
- note added: "Input current limit Resistors ESDA6V1-4BC6 Breakdown Voltage max = 8V ADS131M08 Vin min = -1.6V ADS131M08 Max input current = (-8V + 1.6V)/ 1000R = -6.4mA Within -10mA limit"
- note added: "Not sure this is right! Should it use the source resistance(~50K)?"
- note removed: "Input current limit Resistors PESD2V0Y1BSF Breakdown Voltage max = 3.6V ADS131M08 Vin min = -1.6V ADS131M08 Max input current = (-3.6V + 1.6V)/ 1000R = -2mA Within -10mA limit"
- note removed: "PESD2V0Y1BSF Bidirectional ESD Protection according to IEC 61000-4-2 Reverse Standoff Voltage max = 2V Breakdown Voltage max = 3.6V Capacitance 0.69pF Leakage current max = 50nA"
